Commit message: grasping looks good + fix location

File: config/urdf/stretch_manip_mode.urdf (robot description, URDF)
Before this commit: robot stretch_description, 47 links, 46 joints
Links:
- removed link link_straight_gripper
- added link base_imu, mass 0.00092; collision mesh filename=../meshes/base_imu.STL; visual mesh filename=../meshes/base_imu.STL
- added link link_aruco_d405, mass 0.000393662237156561; collision mesh filename=../meshes/link_SG3_aruco_d405.STL; visual mesh filename=../meshes/link_SG3_aruco_d405.STL
- added link link_aruco_fingertip_left, mass 7.44175884388882E-05; collision mesh filename=../meshes/link_SG3_aruco_fingertip_left.STL; visual mesh filename=../meshes/link_SG3_aruco_fingertip_left.STL
- added link link_aruco_fingertip_right, mass 7.44175884388862E-05; collision mesh filename=../meshes/link_SG3_aruco_fingertip_right.STL; visual mesh filename=../meshes/link_SG3_aruco_fingertip_right.STL
- added link link_grasp_center
- added link link_gripper_s3_body, mass 0.288995995074102; collision mesh filename=../meshes/link_SG3_gripper_body_collision.STL; visual mesh filename=../meshes/link_SG3_gripper_body.STL
- added link link_head_nav_cam, mass 0.028346169831483; collision mesh filename=../meshes/link_SE3_head_nav_cam_collision.STL; visual mesh filename=../meshes/link_SE3_head_nav_cam.STL
- added link link_wrist_quick_connect
- link base_link: mass 1.1912 -> 17.384389; geometry collision mesh filename=../meshes/base_link_collision.STL; visual mesh filename=../meshes/base_link.STL
- link camera_link: geometry collision box size=0.02505 0.09 0.025; visual mesh filename=../meshes/d435.dae
- link laser: mass 0.0749979022894495 -> 0.216007; geometry collision mesh filename=../meshes/laser_collision.STL; visual mesh filename=../meshes/laser.STL
- link link_arm_l0: mass 0.085003260946398 -> 0.427734; geometry collision mesh filename=../meshes/link_arm_l0_collision.STL; visual mesh filename=../meshes/link_arm_l0.STL
- link link_arm_l1: mass 0.051382 -> 0.113658; geometry collision mesh filename=../meshes/link_arm_l1_collision.STL; visual mesh filename=../meshes/link_arm_l1.STL
- link link_arm_l2: mass 0.0571386353275368 -> 0.130565; geometry collision mesh filename=../meshes/link_arm_l2_collision.STL; visual mesh filename=../meshes/link_arm_l2.STL
- link link_arm_l3: mass 0.0628927381893134 -> 0.146817; geometry collision mesh filename=../meshes/link_arm_l3_collision.STL; visual mesh filename=../meshes/link_arm_l3.STL
- link link_arm_l4: mass 0.068095 -> 0.235626; geometry collision mesh filename=../meshes/link_arm_l4_collision.STL; visual mesh filename=../meshes/link_arm_l4.STL
- link link_aruco_inner_wrist: mass 0.0 -> 0
- link link_aruco_left_base: mass 3.59999999990368e-06 -> 3.59999999990368E-06
- link link_aruco_right_base: mass 3.59999999990368e-06 -> 3.59999999990368E-06
- link link_aruco_shoulder: mass 0.0 -> 0
- link link_aruco_top_wrist: mass 0.0 -> 0
- link link_gripper_finger_left: mass 0.0476207785199479 -> 0.0483698266031602; geometry collision mesh filename=../meshes/link_SG3_gripper_finger_left_collision.STL; visual mesh filename=../meshes/link_SG3_gripper_finger_left.STL
- link link_gripper_finger_right: mass 0.047621 -> 0.0483698337858479; geometry collision mesh filename=../meshes/link_SG3_gripper_finger_right_collision.STL; visual mesh filename=../meshes/link_SG3_gripper_finger_right.STL
- link link_gripper_fingertip_left: mass 0.00382160686584851 -> 0.00382162054362131; geometry collision mesh filename=../meshes/link_SG3_gripper_fingertip_left_collision.STL; visual mesh filename=../meshes/link_SG3_gripper_fingertip_left.STL
- link link_gripper_fingertip_right: mass 0.00382160881468841 -> 0.00382162062525088; geometry collision mesh filename=../meshes/link_SG3_gripper_fingertip_right_collision.STL; visual mesh filename=../meshes/link_SG3_gripper_fingertip_right.STL
- link link_head: mass 0.133027236718691 -> 0.681871; geometry collision mesh filename=../meshes/link_head_collision.STL; visual mesh filename=../meshes/link_head.STL
- link link_head_pan: mass 0.0273764496535409 -> 0.062462; geometry collision mesh filename=../meshes/link_head_pan_collision.STL; visual mesh filename=../meshes/link_head_pan.STL
- link link_head_tilt: mass 0.090217113313934 -> 0.283548; geometry collision mesh filename=../meshes/link_head_tilt_collision.STL; visual mesh filename=../meshes/link_head_tilt.STL
- link link_left_wheel: mass 0.0042721 -> 0.20773; geometry collision mesh filename=../meshes/link_left_wheel_collision.STL; visual mesh filename=../meshes/link_left_wheel.STL
- link link_lift: mass 0.27218 -> 1.987167; geometry collision mesh filename=../meshes/link_lift_collision.STL; visual mesh filename=../meshes/link_lift.STL
- link link_mast: mass 1.8285 -> 1.764017; geometry collision mesh filename=../meshes/link_mast_collision.STL; visual mesh filename=../meshes/link_mast.STL
- link link_right_wheel: mass 0.0042721 -> 0.20773; geometry collision mesh filename=../meshes/link_right_wheel_collision.STL; visual mesh filename=../meshes/link_right_wheel.STL
- link link_wrist_pitch: mass 0.0701267146295583 -> 0.116590512374845; geometry collision mesh filename=../meshes/link_DW3_wrist_pitch_collision.STL; visual mesh filename=../meshes/link_DW3_wrist_pitch.STL
- link link_wrist_roll: mass 0.00585666394358811 -> 0.0221916689638078; geometry collision mesh filename=../meshes/link_DW3_wrist_roll_collision.STL; visual mesh filename=../meshes/link_DW3_wrist_roll.STL
- link link_wrist_yaw: mass 0.0404746907425003 -> 0.054422; geometry collision mesh filename=../meshes/link_wrist_yaw_collision.STL; visual mesh filename=../meshes/link_wrist_yaw.STL
- link link_wrist_yaw_bottom: mass 0.0988906816399982 -> 0.144548635554334; geometry collision mesh filename=../meshes/link_DW3_wrist_yaw_bottom_collision.STL; visual mesh filename=../meshes/link_DW3_wrist_yaw_bottom.STL
- link respeaker_base: mass 0.015643 -> 0.025175
Joints:
- removed joint joint_straight_gripper
- added joint joint_aruco_d405: type fixed, parent link_gripper_s3_body, child link_aruco_d405, origin xyz=0 0.0671264013906604 0.0297716109784749 rpy=2.96705999342568 -0.000305721573415565 3.1398588194619, axis 0 0 0
- added joint joint_aruco_fingertip_left: type fixed, parent link_gripper_finger_left, child link_aruco_fingertip_left, origin xyz=0.143934974292929 -0.00436381846064454 -8.58640479230455E-05 rpy=-1.76278254451424 0 0.959931088596885, axis 0 0 0
- added joint joint_aruco_fingertip_right: type fixed, parent link_gripper_finger_right, child link_aruco_fingertip_right, origin xyz=-0.143934974292953 -0.00436381846065068 -8.58640479174944E-05 rpy=-1.76278254451426 0 -0.959931088596862, axis 0 0 0
- added joint joint_base_imu: type fixed, parent base_link, child base_imu, origin xyz=-0.12838 0.0031592 0.1474 rpy=-3.1416 0 -1.5708, axis 0 0 0
- added joint joint_grasp_center: type fixed, parent link_gripper_s3_body, child link_grasp_center, origin xyz=0 0 0.23 rpy=-1.5707963267949 -1.5707963267948 0
- added joint joint_gripper_s3_body: type fixed, parent link_wrist_roll, child link_gripper_s3_body, origin xyz=0 0 0.0209999999993159 rpy=0 0 -3.14159265358975, axis 0 0 0
- added joint joint_head_nav_cam: type fixed, parent link_head_tilt, child link_head_nav_cam, origin xyz=0.0402000000000069 -0.0411729746231231 -0.0245785717313561 rpy=0 1.5707963267949 0, axis 0 0 0
- added joint joint_wrist_quick_connect: type fixed, parent link_wrist_roll, child link_wrist_quick_connect, origin xyz=0 0 0.0085 rpy=1.5708 0 -1.5708, axis 0 0 0
- joint camera_accel_joint: origin xyz=-0.01174 -0.00552 0.0051 rpy=0.0 0.0 0.0 -> xyz=-0.01174 -0.00552 0.0051 rpy=0 0 0
- joint camera_accel_optical_joint: origin xyz=0.0 0.0 0.0 rpy=-1.5707963267948966 0.0 -1.5707963267948966 -> xyz=0 0 0 rpy=-1.5707963267948966 0 -1.5707963267948966
- joint camera_color_joint: origin xyz=0.0 0.015 0.0 rpy=0.0 0.0 0.0 -> xyz=0 0.015 0 rpy=0 0 0
- joint camera_color_optical_joint: origin xyz=0.0 0.0 0.0 rpy=-1.5707963267948966 0.0 -1.5707963267948966 -> xyz=0 0 0 rpy=-1.5707963267948966 0 -1.5707963267948966
- joint camera_depth_joint: origin xyz=0.0 0.0 0.0 rpy=0.0 0.0 0.0 -> xyz=0 0 0 rpy=0 0 0
- joint camera_depth_optical_joint: origin xyz=0.0 0.0 0.0 rpy=-1.5707963267948966 0.0 -1.5707963267948966 -> xyz=0 0 0 rpy=-1.5707963267948966 0 -1.5707963267948966
- joint camera_gyro_joint: origin xyz=-0.01174 -0.00552 0.0051 rpy=0.0 0.0 0.0 -> xyz=-0.01174 -0.00552 0.0051 rpy=0 0 0
- joint camera_gyro_optical_joint: origin xyz=0.0 0.0 0.0 rpy=-1.5707963267948966 0.0 -1.5707963267948966 -> xyz=0 0 0 rpy=-1.5707963267948966 0 -1.5707963267948966
- joint camera_infra1_joint: origin xyz=0.0 0.0 0.0 rpy=0.0 0.0 0.0 -> xyz=0 0.0 0 rpy=0 0 0
- joint camera_infra1_optical_joint: origin xyz=0.0 0.0 0.0 rpy=-1.5707963267948966 0.0 -1.5707963267948966 -> xyz=0 0 0 rpy=-1.5707963267948966 0 -1.5707963267948966
- joint camera_infra2_joint: origin xyz=0.0 -0.05 0.0 rpy=0.0 0.0 0.0 -> xyz=0 -0.05 0 rpy=0 0 0
- joint camera_infra2_optical_joint: origin xyz=0.0 0.0 0.0 rpy=-1.5707963267948966 0.0 -1.5707963267948966 -> xyz=0 0 0 rpy=-1.5707963267948966 0 -1.5707963267948966
- joint camera_joint: origin xyz=0.02802960503838624 -0.007608222297947431 0.018218494141479257 rpy=0.010658876360659654 -0.0022761048951753793 0.018675317090921212 -> xyz=0.03 -0.0122 0.0182 rpy=0.0 0.0 0.0
- joint camera_link_joint: origin xyz=0.010600000000000002 0.0175 0.0125 rpy=0.0 0.0 0.0 -> xyz=0.010600000000000002 0.0175 0.0125 rpy=0 0 0
- joint caster_joint: axis 0.0 0.0 1.0 -> 0 0 1; origin xyz=-0.245 0.0 0.032 rpy=-1.5707963267948966 0.0 0.0 -> xyz=-0.245 0.0 0.032 rpy=-1.5707963267948966 0 0
- joint joint_arm_l0: axis 0.0 0.0 1.0 -> 0 0 1; limit lower=0.0 upper=0.13 effort=100.0 velocity=1.0 -> lower=0.0 upper=0.13 effort=100 velocity=1.0; origin xyz=0.0 0.0 -0.0137499999991968 rpy=7.63746778746202e-30 -3.80121128864402e-15 2.62707547767438e-15 -> xyz=0 0 -0.0137499999991968 rpy=7.63746778746202E-30 -3.80121128864402E-15 2.62707547767438E-15
- joint joint_arm_l1: axis 0.0 0.0 1.0 -> 0 0 1; limit lower=0.0 upper=0.13 effort=100.0 velocity=1.0 -> lower=0.0 upper=0.13 effort=100 velocity=1.0; origin xyz=0.0 0.0 0.0129999999999981 rpy=-7.63746778746202e-30 -7.88860905221012e-31 1.11022302462516e-16 -> xyz=0 0 0.0129999999999981 rpy=-7.63746778746202E-30 -7.88860905221012E-31 1.11022302462516E-16
- joint joint_arm_l2: axis 0.0 0.0 1.0 -> 0 0 1; limit lower=0.0 upper=0.13 effort=100.0 velocity=1.0 -> lower=0.0 upper=0.13 effort=100 velocity=1.0; origin xyz=0.0 0.0 0.013 rpy=0.0 1.57655765344625e-30 -1.66533453693773e-16 -> xyz=0 0 0.013 rpy=0 1.57655765344625E-30 -1.66533453693773E-16
- joint joint_arm_l3: axis 0.0 0.0 1.0 -> 0 0 1; limit lower=0.0 upper=0.13 effort=100.0 velocity=1.0 -> lower=0.0 upper=0.13 effort=100 velocity=1.0; origin xyz=0.0 0.0 0.013 rpy=7.68831233799385e-30 2.36716479416092e-30 2.29652732251143e-17 -> xyz=0 0 0.013 rpy=7.68831233799385E-30 2.36716479416092E-30 2.29652732251143E-17
- joint joint_arm_l4: axis 0.0 0.0 0.0 -> 0 0 0; origin xyz=-0.25956015433181046 -0.0059261537843136765 -0.005557384627505743 rpy=1.5619286973774569 -0.006924580188019336 -1.575847166561953 -> xyz=-0.2547 0 0 rpy=1.5708 2.4721E-15 -1.5708
- joint joint_aruco_inner_wrist: axis 0.0 0.0 0.0 -> 0 0 0; origin xyz=0.0472499999999947 -0.0119000000000034 -0.0272499999991938 rpy=3.14159265358979 4.23377442363088e-14 3.14159265358979 -> xyz=0.0472499999999947 -0.0119000000000034 -0.0272499999991938 rpy=3.14159265358979 4.23377442363088E-14 3.14159265358979
- joint joint_aruco_left_base: axis 0.0 0.0 0.0 -> 0 0 0; origin xyz=-0.00500000000000014 0.1304972 0.1597482 rpy=0.0 0.0 -1.5707963267949 -> xyz=-0.00500000000000014 0.1304972 0.1597482 rpy=0 0 -1.5707963267949
- joint joint_aruco_right_base: axis 0.0 0.0 0.0 -> 0 0 0; origin xyz=-0.0015028 -0.1304972 0.1597482 rpy=0.0 0.0 -1.5707963267949 -> xyz=-0.0015028 -0.1304972 0.1597482 rpy=0 0 -1.5707963267949
- joint joint_aruco_shoulder: axis 0.0 0.0 0.0 -> 0 0 0; origin xyz=-0.0133768876375287 0.0558540528812078 0.0861368272417975 rpy=-1.53998860117704e-29 3.55962409571165e-15 0.0 -> xyz=-0.0133768876375287 0.0558540528812078 0.0861368272417975 rpy=-1.53998860117704E-29 3.55962409571165E-15 0.0
- joint joint_aruco_top_wrist: axis 0.0 0.0 0.0 -> 0 0 0; origin xyz=0.0472500000000019 0.0292850000000015 0.0 rpy=1.5707963267949 -8.03728587323464e-15 3.14159265358979 -> xyz=0.0472500000000019 0.0292850000000015 0 rpy=1.5707963267949 -8.03728587323464E-15 3.14159265358979
- joint joint_gripper_finger_left: axis 0.0 0.0 -1.0 -> 0 0 -1; limit lower=-0.6 upper=0.6 effort=100.0 velocity=1.0 -> lower=0 upper=0 effort=0 velocity=0; origin xyz=0.018599 0.003 0.033689 rpy=1.5708 -1.5708 0.0 -> xyz=0.0245029393015013 0 0.0371909405167127 rpy=-1.57079632679523 -1.48789318734672 -3.14159265358946; parent link_straight_gripper -> link_gripper_s3_body
- joint joint_gripper_finger_right: axis 0.0 0.0 1.0 -> 0 0 1; limit lower=-0.6 upper=0.6 effort=100.0 velocity=1.0 -> lower=0 upper=0 effort=0 velocity=0; origin xyz=-0.018599 0.003 0.033689 rpy=1.5708 1.5708 0.0 -> xyz=-0.0246929393014972 0 0.0371909405167257 rpy=-1.57079632679513 1.48789318732515 3.14159265358956; parent link_straight_gripper -> link_gripper_s3_body
- joint joint_gripper_fingertip_left: axis 0.0 0.0 0.0 -> 0 0 0; origin xyz=0.190596948563868 -0.015 0.0 rpy=1.57079632679496 4.51275387511463e-14 2.60113659715756 -> xyz=0.177784508377884 -0.0106721811879429 0 rpy=1.57079632679491 0 2.87979326579064
- joint joint_gripper_fingertip_right: axis 0.0 0.0 0.0 -> 0 0 0; origin xyz=-0.190596948563868 -0.015 0.0 rpy=-1.57079632679483 -3.43320051448326e-14 0.540456056432235 -> xyz=-0.177784508377902 -0.0106721811879468 0 rpy=-1.5707963267949 0 0.261799387799172
- joint joint_head: axis 0.0 0.0 0.0 -> 0 0 0; origin xyz=0.0 1.33 0.0 rpy=1.5707963267949 -1.5707963267949 3.1416 -> xyz=0 1.33 0 rpy=1.5707963267949 -1.5707963267949 3.1416
- joint joint_head_pan: axis 0.0 0.0 1.0 -> 0 0 1; limit lower=-3.9 upper=1.5 effort=100.0 velocity=1.0 -> lower=-3.9 upper=1.5 effort=100 velocity=1.0; origin xyz=0.1284513021260868 0.07637128403435504 0.00023722543808071166 rpy=-0.013467967166369273 0.005690738105448956 1.6024957766579377 -> xyz=0.135 0.0731000000000001 -0.00319621125547975 rpy=0 0 1.5707963267949
- joint joint_head_tilt: axis 0.0 0.0 1.0 -> 0 0 1; limit lower=-1.53 upper=0.79 effort=100.0 velocity=1.0 -> lower=-1.53 upper=0.79 effort=100 velocity=1.0; origin xyz=0.0032337815907659225 0.030910701770693223 -0.04783143162927699 rpy=1.5763332066189244 -0.029319157204454882 -0.005080558641851002 -> xyz=-0.00130000001785262 0.0277624999926072 -0.0533107920897029 rpy=1.5707963267949 3.36459255518345E-15 -8.42914893687103E-17
- joint joint_laser: axis 0.0 0.0 0.0 -> 0 0 0; origin xyz=0.004 0.0 0.1664 rpy=0.0 0.0 3.1416 -> xyz=0.004 0 0.1664 rpy=0 0 3.1416
- joint joint_left_wheel: axis 0.0 0.0 1.0 -> 0 0 1; origin xyz=0.0 0.17035 0.0508 rpy=-1.5708 2.6317e-16 -8.2057e-19 -> xyz=0 0.17035 0.0508 rpy=-1.5708 2.6317E-16 -8.2057E-19
- joint joint_lift: axis 0.0 0.0 1.0 -> 0 0 1; limit lower=0.0 upper=1.1 effort=100.0 velocity=1.0 -> lower=0.0 upper=1.1 effort=100 velocity=1.0; origin xyz=-0.037385 0.1666 0.0 rpy=-1.5708 1.5708 0.0 -> xyz=-0.037385 0.1666 0 rpy=-1.5708 1.5708 0
- joint joint_mast: axis 0.0 0.0 0.0 -> 0 0 0; origin xyz=-0.07174416574437388 0.13780491000396983 0.03663931715774088 rpy=1.5780076046568878 0.016499709009588637 -0.007971437955302632 -> xyz=-0.067 0.135 0.0284 rpy=1.5708 0 4.8006E-17
- joint joint_respeaker: axis 0.0 0.0 0.0 -> 0 0 0; origin xyz=0.0 1.37236408874452 0.00303065898329655 rpy=-1.5707963267949 -0.698131700797725 4.93295812652799e-16 -> xyz=0 1.37236408874452 0.00303065898329655 rpy=-1.5707963267949 -0.698131700797725 4.93295812652799E-16
- joint joint_right_wheel: axis 0.0 0.0 1.0 -> 0 0 1; origin xyz=0.0 -0.17035 0.0508 rpy=-1.5708 1.2717e-16 4.8006e-17 -> xyz=0 -0.17035 0.0508 rpy=-1.5708 1.2717E-16 4.8006E-17
- joint joint_wrist_pitch: axis 0.0 0.0 -1.0 -> 0 0 -1; limit lower=-1.57 upper=0.56 effort=100.0 velocity=1.0 -> lower=-1.57 upper=0.56 effort=100 velocity=1.0; origin xyz=0.0 -0.0195500000000002 -0.0247499999999984 rpy=1.5707963267949 -8.12895570882604e-15 -3.14159265358979 -> xyz=0 -0.019455 -0.0305 rpy=1.5708 0 3.1416
- joint joint_wrist_roll: axis 0.0 0.0 1.0 -> 0 0 1; limit lower=-3.14 upper=3.14 effort=100.0 velocity=1.0 -> lower=-3.14 upper=3.14 effort=100 velocity=1.0; origin xyz=-0.0188587444076125 -0.0239999999998942 0.01955 rpy=3.14159265358979 1.5707963267949 0.0 -> xyz=-0.018859 -0.024 0.01955 rpy=3.1416 1.5708 0
- joint joint_wrist_yaw: axis 0.0 0.0 -1.0 -> 0 0 -1; limit lower=-1.75 upper=4.0 effort=100.0 velocity=1.0 -> lower=-1.75 upper=4.0 effort=100 velocity=1.0; origin xyz=0.0830000000000654 -0.0307500000000129 0.0 rpy=1.5708 4.2595e-14 2.6415e-15 -> xyz=0.0830000000000654 -0.0307500000000129 0 rpy=-1.5707963267949 0 3.14159265358978
- joint joint_wrist_yaw_bottom: axis 0.0 0.0 0.0 -> 0 0 0; origin xyz=0.0 0.0 0.0 rpy=-3.14159265358979 1.13367999021379e-14 1.57079632679489 -> xyz=0 0 0 rpy=-3.14159265358979 0 -1.5707963267949
