Commit message: Add custom end effector IK solution

File: src/stretch/config/urdf/stretch_manip_mode.urdf (robot description, URDF)
Before this commit: robot stretch, 54 links, 53 joints
Links:
- added link gripper_camera_bottom_screw_frame
- added link gripper_camera_color_frame
- added link gripper_camera_color_optical_frame
- added link gripper_camera_depth_frame
- added link gripper_camera_depth_optical_frame
- added link gripper_camera_infra1_frame
- added link gripper_camera_infra1_optical_frame
- added link gripper_camera_infra2_frame
- added link gripper_camera_infra2_optical_frame
- added link gripper_camera_link, mass 0.072; collision box size=0.023 0.042 0.042; visual mesh filename=./meshes/d405.stl scale=0.001 0.001 0.001
- link base_imu: geometry collision mesh filename=./meshes/base_imu.STL; visual mesh filename=./meshes/base_imu.STL
- link base_link: geometry collision mesh filename=./meshes/base_link_collision.STL; visual mesh filename=./meshes/base_link.STL
- link camera_link: geometry collision box size=0.02505 0.09 0.025; visual mesh filename=./meshes/d435.dae
- link caster_link: geometry collision sphere radius=0.032; visual mesh filename=./meshes/omni_wheel_m.STL
- link laser: geometry collision mesh filename=./meshes/laser_collision.STL; visual mesh filename=./meshes/laser.STL
- link link_arm_l0: geometry collision mesh filename=./meshes/link_arm_l0_collision.STL; visual mesh filename=./meshes/link_arm_l0.STL
- link link_arm_l1: geometry collision mesh filename=./meshes/link_arm_l1_collision.STL; visual mesh filename=./meshes/link_arm_l1.STL
- link link_arm_l2: geometry collision mesh filename=./meshes/link_arm_l2_collision.STL; visual mesh filename=./meshes/link_arm_l2.STL
- link link_arm_l3: geometry collision mesh filename=./meshes/link_arm_l3_collision.STL; visual mesh filename=./meshes/link_arm_l3.STL
- link link_arm_l4: geometry collision mesh filename=./meshes/link_arm_l4_collision.STL; visual mesh filename=./meshes/link_arm_l4.STL
- link link_aruco_d405: geometry collision mesh filename=./meshes/link_SG3_aruco_d405.STL; visual mesh filename=./meshes/link_SG3_aruco_d405.STL
- link link_aruco_fingertip_left: geometry collision mesh filename=./meshes/link_SG3_aruco_fingertip_left.STL; visual mesh filename=./meshes/link_SG3_aruco_fingertip_left.STL
- link link_aruco_fingertip_right: geometry collision mesh filename=./meshes/link_SG3_aruco_fingertip_right.STL; visual mesh filename=./meshes/link_SG3_aruco_fingertip_right.STL
- link link_aruco_inner_wrist: geometry collision mesh filename=./meshes/link_aruco_inner_wrist.STL; visual mesh filename=./meshes/link_aruco_inner_wrist.STL
- link link_aruco_left_base: geometry collision mesh filename=./meshes/link_aruco_left_base.STL; visual mesh filename=./meshes/link_aruco_left_base.STL
- link link_aruco_right_base: geometry collision mesh filename=./meshes/link_aruco_right_base.STL; visual mesh filename=./meshes/link_aruco_right_base.STL
- link link_aruco_shoulder: geometry collision mesh filename=./meshes/link_aruco_shoulder.STL; visual mesh filename=./meshes/link_aruco_shoulder.STL
- link link_aruco_top_wrist: geometry collision mesh filename=./meshes/link_aruco_top_wrist.STL; visual mesh filename=./meshes/link_aruco_top_wrist.STL
- link link_gripper_finger_left: geometry collision mesh filename=./meshes/link_SG3_gripper_finger_left_collision.STL; visual mesh filename=./meshes/link_SG3_gripper_finger_left.STL
- link link_gripper_finger_right: geometry collision mesh filename=./meshes/link_SG3_gripper_finger_right_collision.STL; visual mesh filename=./meshes/link_SG3_gripper_finger_right.STL
- link link_gripper_fingertip_left: geometry collision mesh filename=./meshes/link_SG3_gripper_fingertip_left_collision.STL; visual mesh filename=./meshes/link_SG3_gripper_fingertip_left.STL
- link link_gripper_fingertip_right: geometry collision mesh filename=./meshes/link_SG3_gripper_fingertip_right_collision.STL; visual mesh filename=./meshes/link_SG3_gripper_fingertip_right.STL
- link link_gripper_s3_body: geometry collision mesh filename=./meshes/link_SG3_gripper_body_collision.STL; visual mesh filename=./meshes/link_SG3_gripper_body.STL
- link link_head: geometry collision mesh filename=./meshes/link_head_collision.STL; visual mesh filename=./meshes/link_head.STL
- link link_head_nav_cam: geometry collision mesh filename=./meshes/link_SE3_head_nav_cam_collision.STL; visual mesh filename=./meshes/link_SE3_head_nav_cam.STL
- link link_head_pan: geometry collision mesh filename=./meshes/link_head_pan_collision.STL; visual mesh filename=./meshes/link_head_pan.STL
- link link_head_tilt: geometry collision mesh filename=./meshes/link_head_tilt_collision.STL; visual mesh filename=./meshes/link_head_tilt.STL
- link link_left_wheel: geometry collision mesh filename=./meshes/link_left_wheel_collision.STL; visual mesh filename=./meshes/link_left_wheel.STL
- link link_lift: geometry collision mesh filename=./meshes/link_lift_collision.STL; visual mesh filename=./meshes/link_lift.STL
- link link_mast: geometry collision mesh filename=./meshes/link_mast_collision.STL; visual mesh filename=./meshes/link_mast.STL
- link link_right_wheel: geometry collision mesh filename=./meshes/link_right_wheel_collision.STL; visual mesh filename=./meshes/link_right_wheel.STL
- link link_wrist_pitch: geometry collision mesh filename=./meshes/link_DW3_wrist_pitch_collision.STL; visual mesh filename=./meshes/link_DW3_wrist_pitch.STL
- link link_wrist_roll: geometry collision mesh filename=./meshes/link_DW3_wrist_roll_collision.STL; visual mesh filename=./meshes/link_DW3_wrist_roll.STL
- link link_wrist_yaw: geometry collision mesh filename=./meshes/link_wrist_yaw_collision.STL; visual mesh filename=./meshes/link_wrist_yaw.STL
- link link_wrist_yaw_bottom: geometry collision mesh filename=./meshes/link_DW3_wrist_yaw_bottom_collision.STL; visual mesh filename=./meshes/link_DW3_wrist_yaw_bottom.STL
- link respeaker_base: geometry collision mesh filename=./meshes/respeaker_base.STL; visual mesh filename=./meshes/respeaker_base.STL
Joints:
- added joint gripper_camera_color_joint: type fixed, parent gripper_camera_link, child gripper_camera_color_frame, origin xyz=0 0.0 0 rpy=0 0 0
- added joint gripper_camera_color_optical_joint: type fixed, parent gripper_camera_color_frame, child gripper_camera_color_optical_frame, origin xyz=0 0 0 rpy=-1.5707963267948966 0 -1.5707963267948966
- added joint gripper_camera_depth_joint: type fixed, parent gripper_camera_link, child gripper_camera_depth_frame, origin xyz=0 0 0 rpy=0 0 0
- added joint gripper_camera_depth_optical_joint: type fixed, parent gripper_camera_depth_frame, child gripper_camera_depth_optical_frame, origin xyz=0 0 0 rpy=-1.5707963267948966 0 -1.5707963267948966
- added joint gripper_camera_infra1_joint: type fixed, parent gripper_camera_link, child gripper_camera_infra1_frame, origin xyz=0 0.0 0 rpy=0 0 0
- added joint gripper_camera_infra1_optical_joint: type fixed, parent gripper_camera_infra1_frame, child gripper_camera_infra1_optical_frame, origin xyz=0 0 0 rpy=-1.5707963267948966 0 -1.5707963267948966
- added joint gripper_camera_infra2_joint: type fixed, parent gripper_camera_link, child gripper_camera_infra2_frame, origin xyz=0 -0.018 0 rpy=0 0 0
- added joint gripper_camera_infra2_optical_joint: type fixed, parent gripper_camera_infra2_frame, child gripper_camera_infra2_optical_frame, origin xyz=0 0 0 rpy=-1.5707963267948966 0 -1.5707963267948966
- added joint gripper_camera_joint: type fixed, parent link_gripper_s3_body, child gripper_camera_bottom_screw_frame, origin xyz=0 0.044142 0.042067 rpy=0 -1.3963 -1.5708
- added joint gripper_camera_link_joint: type fixed, parent gripper_camera_bottom_screw_frame, child gripper_camera_link, origin xyz=0.01085 0.009 0.021 rpy=0 0 0
